File: distro.kicad_pcb (KiCad board)
At the start: 2 copper layers, 41 parts, among them J1 SSW-116-02-S-TRA, J2 TSW-106-02-S-TRA, P1 CONN_2X2, P1 MEGAFIT, SW1 M2022LL2W13, SW2 M2022LL2W13, U1 VHE100W, U2 VHB150W, U3 INA139, U4 INA139, U5 INA139

Commit message: Updating layout and component pad configs.
Parts:
- removed the P1 at (156.2, 53.3)
- removed the P1 at (174.0, 53.3)
- removed SW2: M2022LL2W13, switch-M2022LL2W13
- added BT1: BATTERY, BR2032, F.Cu at (196.5, 246.2)
- added C10: 0.1uF, SM0805, F.Cu at (112.6, 164.7)
- added C11: 0.1uF, SM0805, F.Cu at (271.7, 290.1)
- added C12: 0.022uF, SM0805, F.Cu at (177.9, 190.4)
- added C13: 0.022uF, SM0805, F.Cu at (212.3, 290.1)
- added C14: 0.022uF, SM0805, F.Cu at (323.6, 290.1)
- added C15: 0.022uF, SM0805, F.Cu at (171.5, 292.0)
- added C16: 0.022uF, SM0805, F.Cu at (282.8, 290.1)
- added C17: 0.022uF, SM0805, F.Cu at (179.0, 290.1)
- added C18: 0.1uF, SM0805, F.Cu at (177.9, 186.9)
- added C19: 0.1uF, SM0805, F.Cu at (219.7, 290.1)
- added C20: 0.1uF, SM0805, F.Cu at (189.1, 181.6)
- added C21: 0.1uF, SM0805, F.Cu at (223.5, 290.1)
- added C22: 0.1uF, SM0805, F.Cu at (308.7, 290.1)
- added C23: 0.1uF, SM0805, F.Cu at (301.3, 290.1)
- added C24: 0.1uF, SM0805, F.Cu at (305.0, 290.1)
- added C25: 0.1uF, SM0805, F.Cu at (264.2, 290.1)
- added C26: 0.1uF, SM0805, F.Cu at (268.0, 290.1)
- added C27: 0.1uF, SM0805, F.Cu at (201.2, 290.1)
- added C28: 10uF, c_tant_V, F.Cu at (273.5, 278.6)
- added C29: 100uF, SMDHD/VF, F.Cu at (175.0, 141.4)
- added C30: 1uF, SM1206, F.Cu at (119.5, 172.7)
- added C31: 1uF, SM1206, F.Cu at (202.0, 285.5)
- added C32: 10uF, c_tant_V, F.Cu at (179.8, 151.4)
- added C33: 1uF, SM1206, F.Cu at (183.6, 151.4)
- added C34: 0.1uF, SM0805, F.Cu at (208.6, 290.1)
- added C35: 0.1uF, SM0805, F.Cu at (186.4, 290.1)
- added C36: 0.022uF, SM0805, F.Cu at (204.9, 290.1)
- added C37: 1uF, SM1206, F.Cu at (190.1, 285.5)
- added C38: 0.1uF, SM0805, F.Cu at (167.8, 290.1)
- added C39: 47pF, SM0603, F.Cu at (200.8, 291.9)
- added D1: LED Green, LED-0805, F.Cu at (139.4, 169.5)
- added D10: LED Green, LED-0805, F.Cu at (323.9, 285.1)
- added D11: BI_LED, LED_PLCC3, F.Cu at (179.0, 286.7)
- added D2: LED Green, LED-0805, F.Cu at (213.2, 175.6)
- added D3: MB3045S-E3/8W, d2-pak, F.Cu at (171.5, 162.7)
- added D4: BI_LED, LED_PLCC3, F.Cu at (191.1, 189.2)
- added D5: BI_LED, LED_PLCC3, F.Cu at (330.4, 278.7)
- added D6: BI_LED, LED_PLCC3, F.Cu at (165.8, 286.7)
- added D7: BI_LED, LED_PLCC3, F.Cu at (172.4, 286.7)
- added D8: BI_LED, LED_PLCC3, F.Cu at (343.6, 278.7)
- added D9: BI_LED, LED_PLCC3, F.Cu at (323.7, 278.7)
- added F10: 1.1A 5V, littelfuse-1206, F.Cu at (138.1, 123.6)
- added F11: 1.1A 24V, littelfuse-2920L, F.Cu at (258.0, 185.9)
- added F12: 2.6A 5V, littelfuse-1206, F.Cu at (133.0, 188.4)
- added F13: 1.1A 24V, littelfuse-2920L, F.Cu at (168.6, 279.3)
- added F14: 1.1A 5V, littelfuse-1206, F.Cu at (135.6, 194.8)
- added F15: 1.1A 5V, littelfuse-1206, B.Cu at (144.4, 189.7)
- added F16: 1.85A 24V, littelfuse-2920L, F.Cu at (181.4, 279.3)
- added F17: 1.1A 5V, littelfuse-1206, F.Cu at (240.1, 285.5)
- added F18: 1.6A 24V, littelfuse-2920L, F.Cu at (256.6, 272.1)
- added F19: 1.6A 24V, littelfuse-2920L, F.Cu at (295.0, 272.1)
- added F20: 1.1A 24V, littelfuse-2920L, F.Cu at (184.7, 195.9)
- added F21: 1.6A 24V, littelfuse-2920L, F.Cu at (333.4, 272.1)
- added F22: 1.1A 24V, littelfuse-2920L, F.Cu at (195.1, 195.9)
- added F23: 1.6A 24V, littelfuse-2920L, F.Cu at (346.2, 272.1)
- added F24: 1.1A 24V, littelfuse-2920L, F.Cu at (231.1, 272.1)
- added F25: 1.1A 24V, littelfuse-2920L, F.Cu at (218.3, 272.1)
- added F26: 1.1A 24V, littelfuse-2920L, F.Cu at (205.5, 272.1)
- added F27: 1.1A 24V, littelfuse-2920L, F.Cu at (192.7, 272.1)
- added F28: 1.1A 5V, littelfuse-1206, F.Cu at (140.6, 123.6)
- added F29: 1.1A 5V, littelfuse-1206, F.Cu at (230.6, 114.3)
- added F30: 1.5A 5V, littelfuse-1206, F.Cu at (197.2, 114.2)
- added F31: 1.1A 24V, littelfuse-2920L, F.Cu at (282.2, 272.1)
- added F32: 1.1A 24V, littelfuse-2920L, F.Cu at (179.9, 272.1)
- added F33: 1.85A 24V, littelfuse-2920L, F.Cu at (269.4, 272.1)
- added J10: JST-PA-4, s4b-ph-sm4-tb, B.Cu at (146.0, 200.3)
- added J11: JST-PA-2, s2b-ph-sm4-tb, F.Cu at (250.1, 190.3)
- added J12: JST-PA-2, s2b-ph-sm4-tb, F.Cu at (130.5, 201.9)
- added J13: DF13-4, df13-4p-125h, F.Cu at (167.9, 273.5)
- added J14: JST-PA-2, s2b-ph-sm4-tb, B.Cu at (130.5, 200.9)
- added J15: JST-PA-2, s2b-ph-sm4-tb, B.Cu at (219.0, 200.9)
- added J16: JST-PA-2, s2b-ph-sm4-tb, F.Cu at (239.8, 190.1)
- added J17: JST-PA-3, s3b-ph-sm4-tb, F.Cu at (189.9, 201.9)
- added J18: JST-PA-3, s3b-ph-sm4-tb, B.Cu at (188.6, 200.9)
- added J19: JST-PA-4, s4b-ph-sm4-tb, F.Cu at (173.5, 201.9)
- added J20: JST-PA-4, s4b-ph-sm4-tb, B.Cu at (172.2, 200.9)
- added J21: JST-PA-3, s3b-ph-sm4-tb, B.Cu at (204.3, 200.9)
- added J22: JST-PA-3, s3b-ph-sm4-tb, F.Cu at (205.5, 201.9)
- added J23: JST-PA-2, s2b-ph-sm4-tb, F.Cu at (142.4, 201.6)
- added J24: JST-PA-2, s2b-ph-sm4-tb, F.Cu at (250.0, 201.6)
- added J25: JST-PA-2, s2b-ph-sm4-tb, F.Cu at (240.0, 201.8)
- added J26: JST-PA-2, s2b-ph-sm4-tb, F.Cu at (220.1, 201.9)
- added J27: DF13-6, df13-6p-125h, F.Cu at (253.2, 264.0)
- added J3: DF13-6, df13-6p-125h, F.Cu at (131.8, 152.8)
- added J4: DF13-5, df13-5p-125h, F.Cu at (152.1, 152.8)
- added J5: DF13-6, df13-6p-125h, F.Cu at (152.1, 141.4)
- added J6: SSW-116-02-S-TRA, con-samtec-SSW-116-02-S-T-RA, F.Cu at (122.9, 110.4)
- added J7: TSW-106-02-S-TRA, con-samtec-TSW-106-02-S-T-RA, B.Cu at (111.4, 201.1)
- added J8: SSW-108-02-S-D-RA, con-samtec-SSW-108-02-S-D-RA, B.Cu at (209.2, 109.7)
- added J9: SSW-106-02-G-D-RA, con-samtec-SSW-106-02-S-D-RA, B.Cu at (239.7, 109.7)
- added L1: 27nH, inductor_smd_0402, F.Cu at (209.1, 291.6)
- added P1: Pad, 1pin, F.Cu at (254.9, 124.9)
- added P2: SMA RA, sma_90_r300.124.403, F.Cu at (230.4, 209.2)
- added P3: Pad, 1pin, F.Cu at (167.3, 194.8)
- added P4: Pad, 1pin, F.Cu at (105.1, 122.4)
- added P5: Pad, 1pin, F.Cu at (254.9, 194.8)
- added P6: Pad, 1pin, F.Cu at (254.9, 114.8)
- added Q1: IRFZ44, d2-pak, F.Cu at (177.3, 175.8)
- added Q2: IRFZ44, d2-pak, F.Cu at (286.2, 229.1)
- added Q3: IRFZ44, d2-pak, F.Cu at (341.8, 229.1)
- added Q4: IRFZ44, d2-pak, F.Cu at (327.9, 229.1)
- added Q5: IRFZ44, d2-pak, F.Cu at (272.3, 229.1)
- added Q6: IRFZ44, d2-pak, F.Cu at (244.5, 229.1)
- added Q7: IRFZ44, d2-pak, F.Cu at (190.1, 140.6)
- added Q8: IRFZ44, d2-pak, F.Cu at (300.1, 229.1)
- added R13: 150, SM0805, F.Cu at (139.4, 173.4)
- added R14: 4.42k, SM0805, F.Cu at (213.2, 179.4)
- added R15: 470, SM0805, B.Cu at (139.4, 189.7)
- added R16: 100k, SM0805, F.Cu at (143.2, 123.6)
- added R17: 510, SM0805, F.Cu at (327.3, 290.1)
- added R18: 100k, SM0805, F.Cu at (182.7, 290.1)
- added R19: 57.6k, SM0805, F.Cu at (193.8, 290.1)
- added R20: 300, SM0805, F.Cu at (190.1, 290.1)
- added R21: 47.5k, SM0805, F.Cu at (175.8, 190.4)
- added R22: 66.5k, SM0805, F.Cu at (175.3, 290.1)
- added R23: 300, SM0805, F.Cu at (189.1, 185.2)
- added R24: 300, SM0805, F.Cu at (227.2, 290.1)
- added R25: 47.5k, SM0805, F.Cu at (319.9, 290.1)
- added R26: 66.5k, SM0805, F.Cu at (197.5, 290.1)
- added R27: 300, SM0805, F.Cu at (316.2, 290.1)
- added R28: 300, SM0805, F.Cu at (312.4, 290.1)
- added R29: 57.6k, SM0805, F.Cu at (279.1, 290.1)
- added R30: 57.6k, SM0805, F.Cu at (286.5, 290.1)
- added R31: 300, SM0805, F.Cu at (275.4, 290.1)
- added R32: 300, SM0805, F.Cu at (297.6, 290.1)
- added R33: 4.42k, SM0805, F.Cu at (331.0, 290.1)
- added R34: 4.42k, SM0805, F.Cu at (338.4, 290.1)
- added R35: 4.42k, SM0805, F.Cu at (197.5, 292.0)
- added R36: 1M, SM0805, F.Cu at (182.7, 292.0)
- added R37: FILTER, SM0603, F.Cu at (203.7, 291.9)
- added R38: FILTER, SM0603, F.Cu at (206.7, 291.9)
- added R39: 10, SM0805, F.Cu at (171.5, 290.1)
- added U10: 74LS74, so-14, F.Cu at (326.5, 245.8)
- added U11: 74LS74, so-14, F.Cu at (336.3, 245.8)
- added U12: MIC5014, so-8, F.Cu at (312.2, 279.8)
- added U13: MIC5014, so-8, F.Cu at (317.5, 279.8)
- added U14: 74LS74, so-14, F.Cu at (205.2, 279.8)
- added U15: 74LS74, so-14, F.Cu at (214.3, 279.8)
- added U16: MCP601-SOT, SOT23-5, F.Cu at (156.0, 168.6)
- added U17: MCP601-SOT, SOT23-5, F.Cu at (114.0, 160.6)
- added U18: MCP601-SOT, SOT23-5, F.Cu at (317.0, 286.0)
- added U19: MCP601-SOT, SOT23-5, F.Cu at (143.0, 168.6)
- added U20: PQD6-D, PQD6-D, B.Cu at (186.1, 141.0)
- added U21: MS4525DO-DS, DIP-8__300, F.Cu at (218.5, 231.1)
- added U22: 74LS74, so-14, F.Cu at (232.6, 279.8)
- added U23: TC1055, SOT23-5, F.Cu at (310.5, 286.0)
- added U24: NEO-M8, NEO-M8N, F.Cu at (229.4, 178.1)
- added U6: INA139, SOT23-5, F.Cu at (156.9, 172.3)
- added U7: 74LS74, so-14, F.Cu at (241.7, 279.8)
- added U8: MIC5014, so-8, F.Cu at (184.3, 182.4)
- added U9: MIC5014, so-8, F.Cu at (301.6, 279.8)
- C1: value 33uF -> 100uF; footprint SM0805 -> SMDHD/VF
- C2: value C -> 100uF; footprint SM0805 -> SMDHD/VF
- C3: value C -> DNP
- C4: value C -> 10uF; footprint SM0805 -> c_tant_V
- C7, C8: value C -> 0.033uF
- F1, F2, F3, F4, F5, F6, F7, F8: value FUSE -> 4A 5V
- F9: value FUSE -> 1.85A 24V; footprint littelfuse-1206 -> littelfuse-2920L
- J1: value SSW-116-02-S-TRA -> MEGAFIT-4SKT; footprint con-samtec-SSW-116-02-S-T-RA -> molex-MEGAFIT-4SKT-RA
- J2: value TSW-106-02-S-TRA -> DF13-4; footprint con-samtec-TSW-106-02-S-T-RA -> df13-4p-125h
- R1, R2, R3: value R -> DNP
- R10: value LVK25 -> 75k; footprint lvk_resistor-LVK25 -> SM0805
- R11: value R -> 10m; footprint SM0805 -> lvk_resistor-LVK25
- R12: value R -> 100k
- R4: value LVK25 -> DNP; footprint lvk_resistor-LVK25 -> SM0805
- R5: value LVK25R002DER -> 2m
- R9: value R -> 2m; footprint SM0805 -> lvk_resistor-LVK25
- U1: footprint cui-VHE100W -> VHE100W; moved to B.Cu
- U2: value VHB150W -> VQE50W; footprint cui-VHB150W -> VQE50W; moved to B.Cu
- U3: value INA139 -> 74LS74; footprint SOT23-5 -> so-14
- moved R1 442.9 mm to (334.7, 290.1)
- moved R2 375.4 mm to (238.3, 290.1)
- moved F9 365.3 mm to (243.8, 272.1)
- moved U3 263.3 mm to (183.5, 188.8)
- moved R11 262.5 mm to (194.4, 176.4)
- moved U5 258.0 mm to (194.3, 169.7), turned to 180 degrees
- moved R12 256.0 mm to (194.4, 166.6)
- moved C8 254.7 mm to (194.4, 164.6)
- moved J2 245.4 mm to (347.6, 264.0)
- moved R7 239.6 mm to (164.1, 290.1)
- moved C2 239.2 mm to (313.8, 264.1)
- moved C6 237.2 mm to (162.1, 173.2), turned to 90 degrees
- moved R6 235.8 mm to (160.0, 173.2), turned to 90 degrees
- moved C9 235.1 mm to (156.9, 175.1)
- moved R5 228.4 mm to (149.9, 172.3), turned to 270 degrees
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Connections:
- net /Battery/meas_voltage renamed N-0000043
- net /FMAIN7_5V renamed /Pixhawk/FMAIN7_5V
- net /FMAIN8_5V renamed /Pixhawk/FMAIN8_5V
- C1 pad 1: (no net) -> +BATT
- C1 pad 2: (no net) -> GND
- C2 pad 1: (no net) -> +BATT
- C2 pad 2: (no net) -> GND
- C3 pad 1: (no net) -> GND
- C3 pad 2: (no net) -> N-0000022
- C4 pad 1: (no net) -> N-0000027
- C4 pad 2: (no net) -> GND
- C6 pad 1: /Battery/meas_current -> N-0000039
- C7 pad 1: (no net) -> GND
- C7 pad 2: (no net) -> N-0000044
- C8 pad 1: (no net) -> GND
- C8 pad 2: (no net) -> N-0000038
- F1 pad 2: /FMAIN1_5V -> /Pixhawk/FMAIN1_5V
- F2 pad 2: /FMAIN2_5V -> /Pixhawk/FMAIN2_5V
- F3 pad 2: /FMAIN3_5V -> /Pixhawk/FMAIN3_5V
- F4 pad 2: /FMAIN4_5V -> /Pixhawk/FMAIN4_5V
- F5 pad 2: /FMAIN5_5V -> /Pixhawk/FMAIN5_5V
- F6 pad 2: /FMAIN6_5V -> /Pixhawk/FMAIN6_5V
- J1 pad 1: GND -> N-0000046
- J1 pad 2: N-000001 -> N-0000046
- J1 pad 3: (no net) -> GND
- J2 pad 1: GND -> (no net)
- J2 pad 2: /FMAIN1_5V -> N-0000087
- J2 pad 3: (no net) -> N-0000088
- R1 pad 1: (no net) -> N-0000026
- R1 pad 2: (no net) -> N-0000024
- R12 pad 1: (no net) -> GND
- R12 pad 2: (no net) -> N-0000038
- R2 pad 1: (no net) -> GND
- R2 pad 2: (no net) -> N-0000024
- R3 pad 1: (no net) -> N-0000027
- R3 pad 2: (no net) -> N-0000021
- R6 pad 1: /Battery/meas_current -> N-0000039
- SW1 pad GND1: (no net) -> N-0000025
- SW1 pad GND2: (no net) -> N-0000025
- SW1 pad GND3: (no net) -> N-0000025
- SW1 pad GND4: (no net) -> N-0000025
- SW1 pad P1: (no net) -> GND
- SW1 pad P2: (no net) -> /Power/5V_ONOFF
- SW1 pad P4: (no net) -> GND
- SW1 pad P5: (no net) -> /Power/24V_ONOFF
- U3 pad 1: (no net) -> N-00000144
- U3 pad 2: (no net) -> +5V
- U3 pad 3: (no net) -> /Identification Lights/RC_IN
- U3 pad 4: (no net) -> +5V
- U4 pad 1: (no net) -> N-0000044
- U4 pad 2: (no net) -> GND
- U4 pad 3: (no net) -> N-0000020
- U4 pad 5: (no net) -> +5V
- U5 pad 1: /Battery/meas_current -> N-0000038
- U5 pad 3: (no net) -> N-0000016
Other:
- board outline added: 160 x 100.3 mm
- rule pad_to_mask_clearance: 0 -> 0.2
- board text added: "12V"
- board text added: "24V"
- board text added: "5V"

Commit message: Preliminary layout complete.
Parts:
- removed C17, C36: 0.022uF, SM0805
- removed C27, C35: 0.1uF, SM0805
- removed D11, D9: BI_LED, LED_PLCC3
- removed R19, R30: 57.6k, SM0805
- removed R20, R32: 300, SM0805
- removed U15, U22: 74LS74, so-14
- F11, F14, F16, F19, F22, F23, F24, F25, F31, J11, J16, Q1, Q2, Q3, Q4, Q5: moved to B.Cu
- J7: value TSW-106-02-S-TRA -> TSW-108-08-G-T-RA; footprint con-samtec-TSW-106-02-S-T-RA -> con-samtec-TSW-108-02-S-T-RA
- R11, R5, R9: footprint lvk_resistor-LVK25 -> LVK25
- moved J2 262.3 mm to (173.0, 68.2), turned to 180 degrees
- moved D5 214.8 mm to (166.6, 139.8), turned to 90 degrees
- moved F17 207.3 mm to (169.2, 90.7), turned to 270 degrees
- moved U9 190.6 mm to (171.5, 140.5)
- moved F23 189.9 mm to (173.2, 193.8), turned to 90 degrees
- moved J13 188.4 mm to (173.0, 85.2), turned to 180 degrees
- moved R34 186.4 mm to (228.2, 139.8), turned to 270 degrees
- moved D8 183.5 mm to (210.1, 152.8), turned to 270 degrees
- moved R28 181.9 mm to (181.9, 163.4), turned to 180 degrees
- moved C14 181.1 mm to (187.7, 170.4), turned to 180 degrees
- moved J27 181.1 mm to (173.7, 101.3), turned to 180 degrees
- moved R33 181.0 mm to (230.2, 139.8), turned to 270 degrees
- moved R25 179.7 mm to (187.7, 168.4)
- moved R1 178.4 mm to (248.5, 133.9), turned to 270 degrees
- moved U13 177.0 mm to (187.0, 160.2)
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Connections:
- D8 pad 1: N-00000184 (its old number) -> /Payload/Payload_Switched
- J11 pad 1: N-00000171 -> N-00000168
- J15 pad 1: N-00000194 -> N-00000185
- J16 pad 1: N-00000176 (its old number) -> N-00000172
- J22 pad 1: N-00000157 -> N-00000158
- J22 pad 2: N-00000158 -> N-00000157
- J23 pad 1: N-00000195 -> N-00000183
- J24 pad 1: N-00000172 -> N-00000171
- J26 pad 1: N-00000177 (its old number) -> N-00000173
- Q5 pad 1: N-00000184 (its old number) -> /Payload/Payload_Switched
- Q6 pad 1: N-00000185 -> /Payload/Payload_Switched
- Q8 pad 1: N-00000180 (its old number) -> /Payload/Payload_Switched
- U14 pad 9: N-00000184 (its old number) -> /Payload/Payload_Switched
- U21 pad 1: (no net) -> GND
- U21 pad 2: (no net) -> +5V
- U21 pad 3: (no net) -> N-0000088
- U21 pad 4: (no net) -> N-0000087
- U23 pad 1: (no net) -> +5V
- U23 pad 2: (no net) -> GND
- U23 pad 4: (no net) -> N-0000028
- U23 pad 5: (no net) -> +3.3V
- U24 pad 10: (no net) -> GND
- U24 pad 11: (no net) -> N-0000079
- U24 pad 12: (no net) -> GND
- U24 pad 13: (no net) -> GND
- U24 pad 20: (no net) -> N-0000083
- U24 pad 21: (no net) -> N-0000073
- U24 pad 22: (no net) -> N-0000071
- U24 pad 23: (no net) -> +3.3V
- U24 pad 24: (no net) -> GND
- U24 pad 7: (no net) -> GND
- U24 pad 9: (no net) -> N-0000074
- U4 pad 4: (no net) -> N-0000019
