File: lidar.sch (KiCad schematic (older format))
At the start: 3 parts, among them J10 JST-PA-4

Commit message: Finishing bom integration with schematic.
Parts:
- R15: Digikey (none) -> P470CCT-ND
Changed lines of the file:
@@
 LIBS:p_samtec
 LIBS:w_transistor
+LIBS:w_analog
 LIBS:distro-cache
 EELAYER 27 0
@@
 Sheet 7 9
 Title ""
-Date "21 aug 2015"
+Date "22 aug 2015"
 Rev ""
 Comp ""
@@
 F 2 "~" V 2030 2650 30  0000 C CNN
 F 3 "~" H 2100 2650 30  0000 C CNN
+F 4 "P470CCT-ND" V 2100 2650 60  0001 C CNN "Digikey"
 	1    2100 2650
 	1    0    0    -1
